Commit message: refresh

File: src/gazebo_urdf/urdf/robot_diff_learning.xacro (robot description, xacro)
@@ -52,6 +52,15 @@
         <parent link="chassi"/>
         <child link="left_wheel"/>
-        <axis xyz="0.0 1.0 0.0"/>
+        <axis xyz="1.0 0.0 0.0"/> <!--indicate the wheel will rotate in x axis-->
     </joint>
+    <transmission name="trans_left_wheel">
+        <type>transmission_interface/SimpleTransmission</type>
+        <joint name="base_to_left_wheel">
+            <hardwareInterface>hardware_interface/VelocityJointInterface</hardwareInterface>
+        </joint>
+        <actuator name="left_wheel_motor">
+            <mechanicalReduction>1</mechanicalReduction>
+        </actuator>
+	</transmission>
 <!--RIGHT WHEEL-->
     <link name="right_wheel">
@@ -78,5 +87,66 @@
         <parent link="chassi"/>
         <child link="right_wheel"/>
-        <axis xyz="0.0 1.0 0.0"/>
+        <axis xyz="1.0 0.0 0.0"/>  <!--indicate the wheel will rotate in x axis-->
+    </joint>
+    <transmission name="trans_right_wheel">
+        <type>transmission_interface/SimpleTransmission</type>
+        <joint name="base_to_right_wheel">
+            <hardwareInterface>hardware_interface/VelocityJointInterface</hardwareInterface>
+        </joint>
+        <actuator name="right_wheel_motor">
+            <mechanicalReduction>1</mechanicalReduction>
+        </actuator>
+	</transmission>
+<!--PIVOT-->
+    <link name="pivot">
+        <visual>
+            <origin xyz="0 0 0" rpy="3.14 0 0" />
+            <geometry>
+                <mesh filename="package://gazebo_urdf/meshes/pivot.dae" />
+            </geometry>
+        </visual>
+        <collision>
+            <origin xyz="0 0 0" rpy="3.14 0 0" />
+            <geometry>
+                <mesh filename="package://gazebo_urdf/meshes/pivot.dae" />
+            </geometry>
+        </collision>
+        <inertial>
+            <origin xyz="0 0 0" rpy="3.14 0 0"/>
+            <mass value="0.0"/>
+            <inertia ixx="0.0"  ixy="0.0"  ixz="0.0" iyy="0.0" iyz="0.0" izz="0.0" />
+        </inertial>
+    </link>
+    <joint name="pivot_to_chassi" type="fixed">
+        <parent link="chassi"/>
+        <child link="pivot"/>
+        <origin xyz="-0.01500 -0.05000 -0.039500" rpy="0 0 0" />
+        <axis xyz="0.0 0.0 0.0"/>
+    </joint>
+<!--PIVOT_WHEEL-->
+    <link name="pivot_wheel">
+        <visual>
+            <origin xyz="0 0 0" rpy="0 0 0" />
+            <geometry>
+                <mesh filename="package://gazebo_urdf/meshes/ball.dae"/>
+            </geometry>
+        </visual>
+        <collision>
+            <origin xyz="0 0 0" rpy="0 0 0" />
+            <geometry>
+                <mesh filename="package://gazebo_urdf/meshes/ball.dae" />
+            </geometry>
+        </collision>
+        <inertial>
+            <origin xyz="0 0 0" rpy="0 0 0"/>
+            <mass value="0"/>
+            <inertia ixx="0.0"  ixy="0.0"  ixz="0.0" iyy="0.0" iyz="0.0" izz="0.0" />
+        </inertial>
+    </link>
+    <joint name="pivot_to_wheel" type="continuous">
+        <parent link="pivot"/>
+        <child link="pivot_wheel"/>
+        <origin xyz="0.013 0.006 -0.010000" rpy="0 0 0" />
+        <axis xyz="1 1 0" />
     </joint>
 </robot>

Commit message: add inertial

File: src/gazebo_urdf/urdf/robot_diff_learning.xacro (robot description, xacro)
@@ -19,6 +19,6 @@
         <inertial>
             <origin xyz="0.0 0.0 0.0" rpy="0.0 0.0 0.0"/>
-            <mass value="0.0"/>
-            <inertia ixx="0.0" ixy="0.0" ixz="0.0" iyy="0.0" iyz="0.0" izz="0.0"/>
+            <mass value="0.049269"/>
+            <inertia ixx="1.14596769e-4" ixy="-5.431e-11" ixz="-1.451e-11" iyy="2.653e-5" iyz="4.381e-6" izz="1.372e-4"/>
         </inertial>
     </link>
@@ -27,4 +27,5 @@
         <parent link="base_link"/>
         <child link="chassi"/>
+        <axis xyz="0.0 1.0 0.0"/>
     </joint>
 <!--LEFT WHEEL-->
@@ -44,6 +45,6 @@
         <inertial>
             <origin xyz="0.0 0.0 0.0" rpy="0.0 0.0 0.0"/>
-            <mass value="0.0"/>
-            <inertia ixx="0.0" ixy="0.0" ixz="0.0" iyy="0.0" iyz="0.0" izz="0.0"/>
+            <mass value="0.025"/>
+            <inertia ixx="1.564e-5" ixy="1.38055957e-15" ixz="3.31600822e-15" iyy="9.66657107e-6" iyz="-1.38581057e-15" izz="9.66701021e-6"/>
         </inertial>
     </link>
@@ -79,6 +80,6 @@
         <inertial>
             <origin xyz="0.0 0.0 0.0" rpy="0.0 0.0 3.14"/>
-            <mass value="0.0"/>
-            <inertia ixx="0.0" ixy="0.0" ixz="0.0" iyy="0.0" iyz="0.0" izz="0.0"/>
+            <mass value="0.025"/>
+            <inertia ixx="1.564e-5" ixy="1.38055957e-15" ixz="3.31600822e-15" iyy="9.66657107e-6" iyz="-1.38581057e-15" izz="9.66701021e-6"/>
         </inertial>
     </link>
@@ -114,6 +115,6 @@
         <inertial>
             <origin xyz="0 0 0" rpy="3.14 0 0"/>
-            <mass value="0.0"/>
-            <inertia ixx="0.0"  ixy="0.0"  ixz="0.0" iyy="0.0" iyz="0.0" izz="0.0" />
+            <mass value="0.011"/>
+            <inertia ixx="1.812e-6"  ixy="-1.199e-11"  ixz="-4.448e-9" iyy="1.783e-6" iyz="-1.755e-9" izz="9.698e-7" />
         </inertial>
     </link>
@@ -140,6 +141,6 @@
         <inertial>
             <origin xyz="0 0 0" rpy="0 0 0"/>
-            <mass value="0"/>
-            <inertia ixx="0.0"  ixy="0.0"  ixz="0.0" iyy="0.0" iyz="0.0" izz="0.0" />
+            <mass value="0.002"/>
+            <inertia ixx="8.024e-8"  ixy="0.000e+0"  ixz="0.000e+0" iyy="8.024e-8" iyz="1.949e-16" izz="8.320e-8"/>
         </inertial>
     </link>

Commit message: refresh 3.0

File: src/gazebo_urdf/urdf/robot_diff_learning.xacro (robot description, xacro)
@@ -1,4 +1,6 @@
 <?xml version="1.0"?>
 <robot name="robot_diff" xmlns:xacro="http://ros.org/wiki/xacro">
+<!-- Included URDF/XACRO Files -->
+<xacro:include filename="$(find gazebo_urdf)/urdf/rodas.xacro" />
     <link name="base_link">
     </link>
@@ -19,6 +21,6 @@
         <inertial>
             <origin xyz="0.0 0.0 0.0" rpy="0.0 0.0 0.0"/>
-            <mass value="0.049269"/>
-            <inertia ixx="1.14596769e-4" ixy="-5.431e-11" ixz="-1.451e-11" iyy="2.653e-5" iyz="4.381e-6" izz="1.372e-4"/>
+            <mass value="0.074"/>
+            <inertia ixx="1.791e-4" ixy="-2.655e-6" ixz="9.722e-8" iyy="4.091e-5" iyz="5.020e-6" izz="2.027e-4"/>
         </inertial>
     </link>
@@ -30,5 +32,5 @@
     </joint>
 <!--LEFT WHEEL-->
-    <link name="left_wheel">
+    <!-- <link name="left_wheel">
         <visual>
             <origin xyz="0.0 0.0 0.0" rpy="0.0 0.0 0.0"/>
@@ -53,17 +55,23 @@
         <parent link="chassi"/>
         <child link="left_wheel"/>
-        <axis xyz="1.0 0.0 0.0"/> <!--indicate the wheel will rotate in x axis-->
-    </joint>
-    <transmission name="trans_left_wheel">
-        <type>transmission_interface/SimpleTransmission</type>
-        <joint name="base_to_left_wheel">
-            <hardwareInterface>hardware_interface/VelocityJointInterface</hardwareInterface>
-        </joint>
-        <actuator name="left_wheel_motor">
-            <mechanicalReduction>1</mechanicalReduction>
-        </actuator>
-	</transmission>
+        <axis xyz="1.0 0.0 0.0"/> <!-indicate the wheel will rotate in x axis
+    </joint> -->
+<!--
+########################################################################################
+Modelagem das rodas "link" "joint" "transmission" "gazebo"
+########################################################################################
+-->
+    <xacro:robot_diff_wheel side_wheel="left">
+        <origin xyz="0.00 0.0 -0.0" rpy="0 0 0" />
+        <origin xyz="0.048790 0.019314 -0.015708" rpy="0.0 0.0 0.0"/>
+        <origin xyz="0.00 0.0 -0.0" rpy="0 0 0" />
+    </xacro:robot_diff_wheel>
+    <xacro:robot_diff_wheel side_wheel="right">
+        <origin xyz="0.00 -0.00 -0.00" rpy="0 0 3.14" />
+        <origin xyz="-0.048332 0.021179 -0.015706" rpy="0.0 0.0 0.0"/>
+        <origin xyz="0.00 -0.00 -0.00" rpy="0 0 0" />
+    </xacro:robot_diff_wheel>
 <!--RIGHT WHEEL-->
-    <link name="right_wheel">
+ <!-- <link name="right_wheel">
         <visual>
             <origin xyz="0.0 0.0 0.0" rpy="0.0 0.0 3.14"/>
@@ -88,5 +96,5 @@
         <parent link="chassi"/>
         <child link="right_wheel"/>
-        <axis xyz="1.0 0.0 0.0"/>  <!--indicate the wheel will rotate in x axis-->
+        <axis xyz="1.0 0.0 0.0"/>  <indicate the wheel will rotate in x axis
     </joint>
     <transmission name="trans_right_wheel">
@@ -98,7 +106,7 @@
             <mechanicalReduction>1</mechanicalReduction>
         </actuator>
-	</transmission>
+	</transmission> -->
 <!--PIVOT-->
-    <link name="pivot">
+    <!-- <link name="pivot">
         <visual>
             <origin xyz="0 0 0" rpy="3.14 0 0" />
@@ -124,5 +132,5 @@
         <origin xyz="-0.01500 -0.05000 -0.039500" rpy="0 0 0" />
         <axis xyz="0.0 0.0 0.0"/>
-    </joint>
+    </joint>  -->
 <!--PIVOT_WHEEL-->
     <link name="pivot_wheel">
@@ -146,8 +154,36 @@
     </link>
     <joint name="pivot_to_wheel" type="continuous">
-        <parent link="pivot"/>
+        <parent link="chassi"/>
         <child link="pivot_wheel"/>
-        <origin xyz="0.013 0.006 -0.010000" rpy="0 0 0" />
+        <origin xyz="0.00 -0.035 -0.039" rpy="0 0 0" />
         <axis xyz="1 1 0" />
     </joint>
+    <transmission name="trans_wheel" >
+        <type>transmission_interface/SimpleTransmission</type>
+        <joint name="pivot_to_wheel">
+            <hardwareInterface>hardware_interface/EffortJointInterface</hardwareInterface>
+        </joint>
+        <actuator name="act_wheel">
+            <mechanicalReduction>1</mechanicalReduction>
+        </actuator>
+    </transmission>
+    <gazebo reference="pivot_wheel">
+        <mu1 value="100000.0"/>
+        <mu2 value="100.0"/>
+        <kp  value="10000000.0" />
+        <kd  value="1.0" />
+        <fdir1 value="1 0 0"/>
+        <turnGravityOff>false</turnGravityOff>
+    </gazebo>
+<!--
+******************************************************************************************
+ros_control gazebo plugin
+******************************************************************************************
+-->
+    <gazebo>
+        <plugin name="gazebo_ros_control" filename="libgazebo_ros_control.so">
+            <robotNamespace>/</robotNamespace>
+            <legacyModeNS>true</legacyModeNS>
+        </plugin>
+    </gazebo>
 </robot>

Commit message: version 3.0

File: src/gazebo_urdf/urdf/robot_diff_learning.xacro (robot description, xacro)
@@ -31,5 +31,5 @@
         <axis xyz="0.0 1.0 0.0"/>
     </joint>
-<!--LEFT WHEEL-->
+<!--left WHEEL-->
     <!-- <link name="left_wheel">
         <visual>
@@ -62,13 +62,11 @@
 ########################################################################################
 -->
-    <xacro:robot_diff_wheel side_wheel="left">
-        <origin xyz="0.00 0.0 -0.0" rpy="0 0 0" />
-        <origin xyz="0.048790 0.019314 -0.015708" rpy="0.0 0.0 0.0"/>
-        <origin xyz="0.00 0.0 -0.0" rpy="0 0 0" />
+    <xacro:robot_diff_wheel lado_roda="esquerda">
+        <origin xyz="0.049 0.019 -0.016" rpy="0 0 0" />
+        <origin xyz="0 0 0" rpy="0.0 0.0 0.0"/>
     </xacro:robot_diff_wheel>
-    <xacro:robot_diff_wheel side_wheel="right">
-        <origin xyz="0.00 -0.00 -0.00" rpy="0 0 3.14" />
-        <origin xyz="-0.048332 0.021179 -0.015706" rpy="0.0 0.0 0.0"/>
-        <origin xyz="0.00 -0.00 -0.00" rpy="0 0 0" />
+    <xacro:robot_diff_wheel lado_roda="direita">
+        <origin xyz="-0.048 0.021 -0.016" rpy="0 0 0" />
+        <origin xyz="0 0 0" rpy="0.0 0.0 3.14"/>
     </xacro:robot_diff_wheel>
 <!--RIGHT WHEEL-->
@@ -181,9 +179,25 @@
 ******************************************************************************************
 -->
-    <gazebo>
+    <!-- <gazebo>
         <plugin name="gazebo_ros_control" filename="libgazebo_ros_control.so">
             <robotNamespace>/</robotNamespace>
             <legacyModeNS>true</legacyModeNS>
         </plugin>
-    </gazebo>
+    </gazebo> -->
+<!--gazebo diferential drive plugin-->
+  <gazebo>
+    <plugin filename="libgazebo_ros_diff_drive.so" name="differential_drive_controller">
+      <alwaysOn>true</alwaysOn>
+      <updateRate>20</updateRate>
+      <leftJoint>base_to_roda_esquerda</leftJoint>
+      <rightJoint>base_to_roda_direita</rightJoint>
+      <wheelSeparation>0.4</wheelSeparation>
+      <wheelDiameter>0.2</wheelDiameter>
+      <torque>0.1</torque>
+      <commandTopic>cmd_vel</commandTopic>
+      <odometryTopic>odom</odometryTopic>
+      <odometryFrame>odom</odometryFrame>
+      <robotBaseFrame>link_chassis</robotBaseFrame>
+    </plugin>
+  </gazebo>
 </robot>

File: src/gazebo_urdf/urdf/rodas.xacro (robot description, xacro)
@@ -1,5 +1,5 @@
 <?xml version="1.0"?>
 <robot name="robot_diff_wheel" xmlns:xacro="http://ros.org/wiki/xacro" >
-<xacro:macro name="robot_diff_wheel" params="side_wheel *joint_roda_pose *mesh_pose *joint_motor_pose">
+<xacro:macro name="robot_diff_wheel" params="lado_roda *joint_roda_pose *mesh_pose">
 <!--
 ########################################################################################
@@ -7,5 +7,5 @@
 ########################################################################################
 -->
-	<link name="roda_${side_wheel}">
+	<link name="roda_${lado_roda}">
 		<visual>
 			<xacro:insert_block name="mesh_pose"/>
@@ -26,20 +26,20 @@
 		</inertial>
 	</link>
-	<joint name="base_to_roda_${side_wheel}" type="continuous">
+	<joint name="base_to_roda_${lado_roda}" type="continuous">
 		<parent link="chassi"/>
-		<child link="roda_${side_wheel}"/>
+		<child link="roda_${lado_roda}"/>
 		<xacro:insert_block name="joint_roda_pose"/>
 		<axis xyz="1 0 0" rpy="0 0 0" />
 	</joint>
-	<transmission name="trans_roda_${side_wheel}">
+	<transmission name="trans_roda_${lado_roda}">
 		<type>transmission_interface/SimpleTransmission</type>
-		<joint name="base_to_roda_${side_wheel}">
+		<joint name="base_to_roda_${lado_roda}">
 			<hardwareInterface>hardware_interface/VelocityJointInterface</hardwareInterface>
 		</joint>
-		<actuator name="roda_${side_wheel}_motor">
+		<actuator name="roda_${lado_roda}_motor">
 			<mechanicalReduction>1</mechanicalReduction>
 		</actuator>
 	</transmission>
-	<gazebo reference="roda_${side_wheel}">
+	<gazebo reference="roda_${lado_roda}">
 		<mu1 value="1.0"/>
 		<mu2 value="1.0"/>
@@ -48,33 +48,4 @@
 		<fdir1 value="1 0 0"/>
 	</gazebo>
-<!--
-########################################################################################
-Modelagem da motor direita "link" "joint"
-########################################################################################
--->
-	<link name="motor_${side_wheel}">
-		<visual>
-			<origin xyz="0 0 0" rpy="0 0 0" />
-			<geometry>
-				<mesh filename="package://gazebo_urdf/meshes/Roue_65mm.dae" />
-			</geometry>
-		</visual>
-		<collision>
-			<origin xyz="0 0 0" rpy="0 0 0" />
-			<geometry>
-				<mesh filename="package://gazebo_urdf/meshes/Roue_65mm.dae" />
-			</geometry>
-		</collision>
-		<inertial>
-			<origin xyz="0 0 0" rpy="0 0 0"/>
-			<mass value="0.025"/>
-			<inertia ixx="1.564e-5" ixy="1.38055957e-15" ixz="3.31600822e-15" iyy="9.66657107e-6" iyz="-1.38581057e-15" izz="9.66701021e-6" />
-		</inertial>
-	</link>
-	<joint name="base_to_motor_${side_wheel}" type="fixed">
-		<parent link="chassi"/>
-		<child link="motor_${side_wheel}"/>
-		<xacro:insert_block name="joint_motor_pose"/>
-	</joint>
 </xacro:macro>
 </robot>
